Commit message: [1.0.3] Updating Files from the original package to fix RVIZ TF issues

File: urdf/domain.xacro (robot description, xacro)
@@ -424,3 +424,17 @@
     </transmission>
   </xacro:macro>
+  <!-- Create a camera link and its child optical link. -->
+  <xacro:macro
+    name="camera_link"
+    params="name"
+  >
+    <link name="${name}"/>
+    <link name="${name}_optical"/>
+    <xacro:joint_fixed
+      parent="${name}"
+      child="${name}_optical"
+      roll="${-0.5 * pi}"
+      yaw="${-0.5 * pi}"
+    />
+  </xacro:macro>
 </robot>

File: urdf/gazebo.xacro (robot description, xacro)
@@ -46,5 +46,5 @@
           <camera_name>${name}</camera_name>
           <!-- Set TF frame name. If empty, defaults to link name (i.e. "link_name") -->
-          <frame_name>${name}</frame_name>
+          <frame_name>${name}_optical</frame_name>
           <hack_baseline>0.07</hack_baseline>
           <!-- No need to repeat distortion parameters or to set autoDistortion -->
@@ -106,7 +106,12 @@
       wheel_diameter
       wheel_separation
+      publish_odom:=false
     "
   >
     <gazebo>
+      <plugin name="${name}_joint_states" filename="libgazebo_ros_joint_state_publisher.so">
+        <joint_name>${right_joint}</joint_name>
+        <joint_name>${left_joint}</joint_name>
+      </plugin>
       <plugin name="${name}_controller" filename="libgazebo_ros_diff_drive.so">
         <update_rate>50</update_rate>
@@ -117,12 +122,8 @@
         <max_wheel_torque>20</max_wheel_torque>
         <max_wheel_acceleration>1.0</max_wheel_acceleration>
-        <command_topic>cmd_vel</command_topic>
-        <odometry_topic>odom</odometry_topic>
         <odometry_frame>odom</odometry_frame>
         <robot_base_frame>base_link</robot_base_frame>
-        <publish_odom>true</publish_odom>
-        <publish_odom_tf>true</publish_odom_tf>
-        <publish_wheel_tf>false</publish_wheel_tf>
-        <publish_wheel_joint_state>true</publish_wheel_joint_state>
+        <publish_odom>${publish_odom}</publish_odom>
+        <publish_odom_tf>${publish_odom}</publish_odom_tf>
       </plugin>
     </gazebo>
